File: pico2_trace.kicad_sch (KiCad schematic)
At the start: 48 parts, among them J1B BREAKOUT, J2B BREAKOUT, J3 MIPI-20, J4 JST-SH-3 DEBUG, J5 USB-A HOST, J6 CORTEX-10, J7 JST-SH-3 DEBUG_PROBE, J8 USB-MICROB PWR, J9 USB-MICROB DEV, SW1 RESET

Commit message: model: realize DNP parts (INA219 opt), EN pulldown, cap ratings, J9_VBUS class
- Add R_HVEN_PD (100k, HOST_VBUS_EN->GND): RP2350-E9 makes the chip's own
  internal pull-downs unreliable before firmware runs, so the TPS2051B EN
  pin needs a real external pulldown to default the host load switch off
  at boot.
- Capacitor values now carry voltage ratings (Adafruit schematic rule):
  C_HVBUS_BULK 22u -> 22u/10V, C_HVBUS_100n/C_NRESET 100n -> 100n/16V.
- Realize the DNP parts Adafruit-style (real footprint + fully wired +
  dnp=True, instead of a stand-in footprint with all pins no-connect):
  U_INA219_ALT gets the real INA219 SOT-23-8 footprint/padmap (TI SBOS448
  Fig 8-1) and is wired across the same shunt as U_ISNS, on the shared
  I2C0 bus, address 0x40. D_J9_BUSPWR/J_TRACE_TP were already wired.
  emit_netlist, gen_sch.py, and build_board.py now include/place/wire DNP
  parts instead of omitting them (KiCad 9 dnp=yes symbol attribute;
  FP_DNP + FP_EXCLUDE_FROM_POS_FILES footprint attribute, still shown in
  BOM). They land at (0,0) for now -- a follow-up compaction/placement
  pass places them for real.
- Add J9_VBUS to the Power netclass pattern list (missing since Task 14).
- docs/PARTS.md: the three Adafruit-component-reuse evaluations (TPS2051B
  kept over AP22802, USBLC6-2SC6 kept over PRTR5V0U2X, INA219 adopted as
  a populatable DNP option), an LCSC-first sourcing note, and a Samtec
  FTSH <-> LCSC keyed-shroud alternate note for the debug headers.

Verified: 7/7 model tests, ERC 0 errors (67 pre-existing off-grid
warnings, unchanged), schematic/reference netlist parity match (DNP nodes
included on both sides), board rebuild idempotent. No geometry changed:
0 of 52 existing footprints moved and the Task 13/14 trace bundle is
byte-identical -- confirmed programmatically, not just by inspection.
Parts:
- added C_NRESET: 100n/16V, Capacitor_SMD:C_0402_1005Metric, symbol gen:GEN2
- added D_J9_BUSPWR: 1N4148W, Diode_SMD:D_SOD-123, symbol gen:GEN2
- added J_TRACE_TP: TRACE_TP, Connector_PinHeader_2.54mm:PinHeader_1x06_P2.54mm_Vertical, symbol gen:GEN6
- added R_HVEN_PD: 100k, Resistor_SMD:R_0402_1005Metric, symbol gen:GEN2
- added U_INA219_ALT: INA219, Package_TO_SOT_SMD:SOT-23-8, symbol gen:GEN8
- C_HVBUS_100n: value 100n -> 100n/16V
- C_HVBUS_BULK: value 22u -> 22u/10V
Connections:
- net GND: now also C_NRESET.2, J_TRACE_TP.6, R_HVEN_PD.2, U_INA219_ALT.3, U_INA219_ALT.7, U_INA219_ALT.8
- net HOST_5V_IN: now also U_INA219_ALT.2
- net HOST_VBUS_EN: now also R_HVEN_PD.1
- net I2C0_SCL: now also U_INA219_ALT.5
- net I2C0_SDA: now also U_INA219_ALT.6
- net J9_VBUS: now also D_J9_BUSPWR.1
- net NRESET: now also C_NRESET.1
- net P3V3: now also U_INA219_ALT.4
- net TD0: now also J_TRACE_TP.2
- net TD1: now also J_TRACE_TP.3
- net TD2: now also J_TRACE_TP.4
- net TD3: now also J_TRACE_TP.5
- net TRACECLK: now also J_TRACE_TP.1
- net VBUS_NET: now also D_J9_BUSPWR.2
- net VBUS_SEL: now also U_INA219_ALT.1

Commit message: lib: blind-bottom SMT sockets (stock land pattern, no through-holes)
Parts:
- removed J_TRACE_TP: TRACE_TP, Connector_PinHeader_2.54mm:PinHeader_1x06_P2.54mm_Vertical, symbol gen:GEN6
- J1B, J2B: footprint Connector_PinSocket_2.54mm:PinSocket_1x20_P2.54mm_Vertical -> Connector_PinSocket_2.54mm:PinSocket_1x20_P2.54mm_Vertical_SMD_Pin1Left
- J5: footprint Connector_USB:USB_A_Molex_67643_Horizontal -> Connector_USB:USB_A_Receptacle_GCT_USB1046
- JP1, J_UART: footprint Connector_PinHeader_2.54mm:PinHeader_1x03_P2.54mm_Vertical -> Connector_PinHeader_2.54mm:PinHeader_1x03_P2.54mm_Vertical_SMD_Pin1Left
- JP2, JP3, JP4: footprint Connector_PinHeader_2.54mm:PinHeader_1x02_P2.54mm_Vertical -> Connector_PinHeader_2.54mm:PinHeader_1x02_P2.54mm_Vertical_SMD_Pin1Left
- PICO: footprint Module:RaspberryPi_Pico_Common_THT -> pico2_trace:PicoSocket_2x20_SMD

Commit message: pcb: revert hand-inserted connectors to THT, re-place, relocate guards
Parts that take repeated hand-insertion force stay through-hole; everything
else stays SMT. Reverts pico_socket/breakout_1x20/hdr_1x02/hdr_1x03/hdr_1x06
to stock THT footprints, retires the custom SMD Pico-socket land pattern
(never itself a traced, orderable part -- the project's largest remaining
fab risk), and re-places J1B/J2B/JP1-4/J_UART against the reverted
footprints' pin-1 anchors. JP2/JP3 (GP0/GP6 guard jumpers) move back into
the J1B->debug-row gap, now that THT J1B's courtyard is slim enough to fit
them -- guard-trace runs to PICO shrink from 42-50mm to ~11.4mm each.

Rt1-5, the debug row, and every cluster outside PICO's own footprint are
unchanged (not PICO-grid-dependent). Breakout pad alignment verified exact
(0.000mm error, all 40 J1B/J2B<->PICO pairs) by construction: both parts
share PICO's 2.54mm pitch and pad-1-first numbering.

Regenerated pico2_trace.net/.kicad_sch/docs/schematic.pdf (embedded
footprint names); netlists match, ERC 0 errors. DRC: 2 pre-existing
silk_edge_clearance violations only (PICO's own edge overhang, a Task 11
decision), courtyards_overlap/holes_co_located/silk_overlap/silk_over_copper
all 0. No routing performed (placement only).
Parts:
- J1B, J2B: footprint Connector_PinSocket_2.54mm:PinSocket_1x20_P2.54mm_Vertical_SMD_Pin1Left -> Connector_PinSocket_2.54mm:PinSocket_1x20_P2.54mm_Vertical
- JP1, J_UART: footprint Connector_PinHeader_2.54mm:PinHeader_1x03_P2.54mm_Vertical_SMD_Pin1Left -> Connector_PinHeader_2.54mm:PinHeader_1x03_P2.54mm_Vertical
- JP2, JP3, JP4: footprint Connector_PinHeader_2.54mm:PinHeader_1x02_P2.54mm_Vertical_SMD_Pin1Left -> Connector_PinHeader_2.54mm:PinHeader_1x02_P2.54mm_Vertical
- PICO: footprint pico2_trace:PicoSocket_2x20_SMD -> Module:RaspberryPi_Pico_Common_THT

Commit message: pcb: add J10 SWD dupont, clear antenna keepout, complete routing
Parts:
- added J10: SWD, Connector_PinHeader_2.54mm:PinHeader_1x03_P2.54mm_Vertical, symbol gen:GEN3
Connections:
- net GND: now also J10.2
- net SWCLK: now also J10.1
- net SWDIO: now also J10.3

Commit message: pcb: remove redundant J4, widen power traces off the pitch crossings
Parts:
- removed J4: JST-SH-3 DEBUG, Connector_JST:JST_SH_SM03B-SRSS-TB_1x03-1MP_P1.00mm_Horizontal, symbol gen:GEN3

Commit message: pcb: fix diode direction, ground J5 shell, add VSYS feed + decoupling, widen V5_JTRACE
Parts:
- removed J5: USB-A HOST, Connector_USB:USB_A_Receptacle_GCT_USB1046, symbol gen:GEN4
- added C_HSW_IN, C_P3V3_1, C_P3V3_2: 100n/16V, Capacitor_SMD:C_0402_1005Metric, symbol gen:GEN2
- added D_VSYS: B5819W, Diode_SMD:D_SOD-123, symbol gen:GEN2
- added J5: USB-A HOST, Connector_USB:USB_A_Receptacle_GCT_USB1046, symbol gen:GEN5
Connections:
- net GND: now also C_HSW_IN.2, C_P3V3_1.2, C_P3V3_2.2, J5.4, J5.5
- net HOST_5V_IN: now also C_HSW_IN.1
- net HOST_DM: now also J5.2
- net HOST_DP: now also J5.3
- net HOST_VBUS: now also J5.1
- net J9_VBUS: now also D_J9_BUSPWR.2; no longer D_J9_BUSPWR.1
- net P3V3: now also C_P3V3_1.1, C_P3V3_2.1
- net VBUS_NET: now also D_J9_BUSPWR.1; no longer D_J9_BUSPWR.2
- net VBUS_SEL: now also D_VSYS.2
- net VSYS: now also D_VSYS.1

Commit message: pcb: J8 micro-B -> USB Type-C power input (C165948) + CC pull-downs
- usb_c_pwr footprint: local renumbered copy of the stock HRO
  TYPE-C-31-M-12 land (1=VBUS A4/B9, 2=CC1, 3=CC2, 4=GND, 5=NC data/SBU,
  6=shield, 7=VBUS A9/B4 second column, board-NC: the NPTH peg blocks
  every legal escape; the plug parallels all four VBUS beams)
- R_CC1/R_CC2 5.1k Rd (C25905) west of the connector; CC stubs run
  north out of the pad row and west under the body (crossing-free lane
  pair y=5.25/5.7, DRC-derived)
- VBUS_NET approach corridor moved y=7.5 -> 5.0 (old lane is under the
  new pad row); pour stitch via (22.0,6.0) -> (23.6,6.9)
- board regenerated from scratch (pipeline first proven byte-equivalent
  vs the frozen 6d67559 board); gates: DRC 0 unconnected + 2 known silk
  warnings, ERC warnings-only, netlists match, pour union-find = 1
  component, checks 7/7
- BOM/BOM_jlc/CPL_jlc/DESIGN/ORDERING updated; new fab zip
Parts:
- removed J8: USB-MICROB PWR, Connector_USB:USB_Micro-B_Molex_47346-0001, symbol gen:GEN6
- added J8: USB-C PWR, pico2_trace:USB_C_PWR_HRO_TYPE-C-31-M-12, symbol gen:GEN7
- added R_CC1, R_CC2: 5.1k, Resistor_SMD:R_0402_1005Metric, symbol gen:GEN2
Connections:
- net GND: now also J8.4, J8.6, R_CC1.2, R_CC2.2
- net VBUS_NET: now also J8.1
- new net J8_CC1: J8.2, R_CC1.1
- new net J8_CC2: J8.3, R_CC2.1
- no-connect marks 10 -> 9

Commit message: pcb: J9 micro-B -> USB Type-C device port (C165948) + CC pull-downs
- usb_c_dev footprint: renumbered HRO land for a USB2 device (1=VBUS,
  2/3=CC, 4=GND, 5=D+ A6/B6, 6=D- A7/B7, 7=SBU nc, 8=second VBUS column
  board-NC, 9=shield)
- interleaved D+/D- pairs bridged with a two-layer weave (D- rail on F,
  D+ through B via pair threading the NPTH peg gap)
- R_CC3/R_CC4 Rd + the VBUS-detect divider relocated to the south band;
  DEV_VBUS_DET tail re-derived (east B_Cu descent at x=86.2); J9_VBUS
  web rebuilt (spine y=54.4, ESD_D.5 tap around the DM wall on B_Cu)
- pour: 1 stale fragment via moved, 2 new stitch vias for the boxed-in
  R_CC4.2/R_J9VD_B.2 ground pockets
- gates: DRC 0 unconnected + 2 baseline silk warnings, checks 7/7, ERC
  warnings-only, netlists match, pour union-find 1 component (39 islands,
  75 vias)
- last micro-B eliminated: C132560 drops from the BOM entirely
Parts:
- removed J9: USB-MICROB DEV, Connector_USB:USB_Micro-B_Molex_47346-0001, symbol gen:GEN6
- added J9: USB-C DEV, pico2_trace:USB_C_DEV_HRO_TYPE-C-31-M-12, symbol gen:GEN9
- added R_CC3, R_CC4: 5.1k, Resistor_SMD:R_0402_1005Metric, symbol gen:GEN2
Connections:
- net DEV_DM: now also J9.6
- net DEV_DP: now also J9.5
- net GND: now also J9.4, J9.9, R_CC3.2, R_CC4.2
- net J9_VBUS: now also J9.1
- new net J9_CC1: J9.2, R_CC3.1
- new net J9_CC2: J9.3, R_CC4.1
- no-connect marks 9 -> 10
