File: pico2_trace_motherboard/pico2_trace.kicad_sch (KiCad schematic)
At the start: 53 parts, among them J1B BREAKOUT, J2B BREAKOUT, J3 MIPI-20, J4 JST-SH-3 DEBUG, J5 USB-A HOST, J6 CORTEX-10, J7 JST-SH-3 DEBUG_PROBE, J8 USB-MICROB PWR, J9 USB-MICROB DEV, SW1 RESET

Commit message: pcb: compact to 92x64; SMT-socket detour reverted to THT
Co-designed placement + routing rewrite; hand-inserted connectors back
to THT after the SMD experiment. Squash of 4fb3f47..d5493a2 (5).
Parts:
- removed J_TRACE_TP: TRACE_TP, Connector_PinHeader_2.54mm:PinHeader_1x06_P2.54mm_Vertical, symbol gen:GEN6
- J5: footprint Connector_USB:USB_A_Molex_67643_Horizontal -> Connector_USB:USB_A_Receptacle_GCT_USB1046

Commit message: pcb: complete routing, GND pours + stitching, power widening
All copper 0 non-GND unconnected; J10 SWD dupont added, redundant J4
removed, antenna keepout cleared; VBUS_NET widened; both-layer GND
zones + stitching vias. Squash of 0dd589d, 7224fb8, 98ee5bf, 9fa26b4.
Parts:
- removed J4: JST-SH-3 DEBUG, Connector_JST:JST_SH_SM03B-SRSS-TB_1x03-1MP_P1.00mm_Horizontal, symbol gen:GEN3
- added J10: SWD, Connector_PinHeader_2.54mm:PinHeader_1x03_P2.54mm_Vertical, symbol gen:GEN3
Connections:
- net GND: now also J10.2
- net SWCLK: now also J10.1
- net SWDIO: now also J10.3
