File: pico2_trace_motherboard/pico2_trace.kicad_pcb (KiCad board)
At the start: 2 copper layers, 92 x 64 mm, 64 parts, among them J10 SWD, J1B BREAKOUT, J2B BREAKOUT, J3 MIPI-20, J5 USB-A HOST, J6 CORTEX-10, J7 JST-SH-3 DEBUG_PROBE, J8 USB-C PWR, J9 USB-C DEV, SW1 RESET

Commit message: pcb(revb): J5 USB-A mouth flush to the board edge + edge-mouth guard
REV A (fabricated, tag rev-a-pico2) shipped with J5's USB-A opening
recessed 6.61mm inside the x=92 edge -- a cable overmold fouls on the
ledge in front of it. Its anchor came from the pad rows and the
mouth-to-edge dimension was never asserted; J8/J9 had explicit flush-lip
arithmetic, J5 predated that convention.

- place.py: J5 anchor 78.615 -> 85.225 (mouth now exactly 92.00);
  BOARD_REV_TEXT REV A -> REV B so the two are distinguishable in hand
- pour.py: stitch via (78.0,22.0) -> (75.0,26.0), 1.0mm from J5's
  relocated HOST_DM pad (DRC clearance + hole_clearance)
- checks.py: new test_edge_connector_mouths asserts every edge-facing
  receptacle's F.Fab mouth is within 1.0mm of its edge; proven
  non-vacuous (fires on REV A's J5 at 6.61mm, passes J8/J9 at 0.45mm)
- docs/REVB_NOTES.md: the fix, the REV A field-rescue notch, and the
  real cost levers (board area saves $0 -- assembly qty and
  Extended->Basic swaps are where the money is)
- fab/MANIFEST.txt: notes the tree has advanced past the ordered REV A

Semantic diff vs rev-a-pico2: J5 moved, 7 tracks on HOST_DP/DM/VBUS,
1 via, REV silk -- nothing else. Gates: DRC 0 unconnected + the 2
baseline silk warnings, checks 8/8, netlists match, pour union-find 1
component (39 islands / 75 vias).
Parts:
- moved J5 6.61 mm to (85.2, 20.0)
Routing:
- net HOST_VBUS: track 32.1 -> 45.3 mm
- net HOST_DM: track 15.5 -> 22.1 mm
- net HOST_DP: track 15.5 -> 22.1 mm
Other:
- board text added: "REV B"
- board text removed: "REV A"
